Commit message: phase_1_tests

File: src/rbot/robot/rlai_description/urdf/control/ros2_control.urdf.xacro (robot description, xacro)
@@ -54,4 +54,12 @@
       <xacro:caster_state_interfaces name="rear_left"/>
       <xacro:caster_state_interfaces name="rear_right"/>
+      <joint name="fork_lift_joint">
+        <command_interface name="velocity">
+          <param name="min">-0.08</param>
+          <param name="max">0.08</param>
+        </command_interface>
+        <state_interface name="position"/>
+        <state_interface name="velocity"/>
+      </joint>
     </ros2_control>
   </xacro:macro>

File: src/rbot/robot/rlai_description/urdf/robot.urdf.xacro (robot description, xacro)
@@ -18,4 +18,5 @@
   <xacro:include filename="$(find rlai_description)/urdf/base/wheels.urdf.xacro"/>
   <xacro:include filename="$(find rlai_description)/urdf/base/payload_platform.urdf.xacro"/>
+  <xacro:include filename="$(find rlai_description)/urdf/base/fork.urdf.xacro"/>
   <xacro:include filename="$(find rlai_description)/urdf/sensors/imu.urdf.xacro"/>
   <xacro:include filename="$(find rlai_description)/urdf/sensors/lidar_2d.urdf.xacro"/>
@@ -71,4 +72,5 @@
   </xacro:if>
   <xacro:rlai_payload_platform parent="base_link"/>
+  <xacro:rlai_fork parent="base_link"/>
   <xacro:rlai_ros2_control sim_mode="$(arg sim_mode)"/>
 </robot>
